File: elec/C3IRuler2026PCB/alimentation.kicad_sch (KiCad schematic)
At the start: 0 parts

Commit message: Trying to get the simulation of square wave working
Parts:
- added R4, R5: 10k, symbol Device:R
- added V2: 10, symbol Simulation_SPICE:VDC
Connections:
- new net -5V: R5.2, V2.2
- new net 0: R4.2, R5.1
- new net 5V: R4.1, V2.1
Other:
- note added: "10V to +/- 5V"
